File: hw/ArcFaultPCB/ArcFaultPCB.kicad_sch (KiCad schematic)
At the start: 15 parts, among them IC2 TS3021AILT, IC3 TLV3602DGKR, IC4 ESP32-WROOM-32E-N4, J2 Conn_01x04_Socket, J3 Conn_01x10_Socket, J4 Conn_01x04_Socket, SW1 SW_Reset

Commit message: arc fault detection schematic mock up
Parts:
- added C2: 18.4nF, symbol Device:C
- added C3, C4, C5: 1uF, symbol Device:C
- added F1: Fuse, symbol Device:Fuse
- added IC1: TS3021AILT, SOT95P280X145-5N, symbol TS3021AILT:TS3021AILT
- added L1: L, symbol Device:L
- added R1: 39.2, symbol Device:R
- added R2: 118, symbol Device:R
- added R3: 13.7, symbol Device:R
- added R4, R5: 3.32k, symbol Device:R
Connections:
- net +3V3: now also C2.1, C5.1, IC1.5 (VCC+), R4.1
- net GND: now also C4.2, C5.2, F1.2, IC1.2 (VCC-), R5.2
- new net: IC1.1 (OUT), R3.1
- new net: IC1.4 (IN-), R2.1, R3.2
- new net: C4.1, IC1.3 (IN+), R4.2, R5.1
- new net: C2.2, L1.1
- new net: F1.1, R1.2
- new net: C3.1, R2.2
- new net: C3.2, L1.2, R1.1
Other:
- moved on the sheet: 3V3, 5V1, AMP_OUT1, C1, DAC_OUT1, J2, J3, J4, POT_OUT1, R10, R9, SW1
